File: Hardware/Production/Qwiic_GPIO-Panel.brd (EAGLE design)
At the start: 186.7 x 167.6 mm, 1027 parts, among them J13 SMD, J14 PTH, J15 SMD, J19 SMD, J2 SMD, J20 PTH, J21 SMD, J25 SMD, J26 PTH, J27 SMD, J3 PTH, J31 SMD, J32 PTH, J33 SMD, J37 SMD, J38 PTH, J39 SMD, J4 SMD, J43 SMD, J44 PTH, J45 SMD, J49 SMD, J50 PTH, J51 SMD, J55 SMD, J56 PTH, J57 SMD, J61 SMD, J62 PTH, J63 SMD, J67 SMD, J68 PTH, J69 SMD, J7 SMD, J73 SMD, J74 PTH, J75 SMD, J79 SMD, J8 PTH, J80 PTH, J81 SMD, J85 SMD, J86 PTH, J87 SMD, J9 SMD, J91 SMD, J92 PTH, J93 SMD, U1 TCA9534U, U10 TCA9534U, U11 TCA9534U, U12 TCA9534U, U13 TCA9534U, U14 TCA9534U, U15 TCA9534U, U16 TCA9534U, U2 TCA9534U, U3 TCA9534U, U4 TCA9534U, U5 TCA9534U, U6 TCA9534U, U7 TCA9534U, U8 TCA9534U, U9 TCA9534U

Commit message: Generated new panel file
Parts:
- added 3V1, 3V10, 3V11, 3V12, 3V13, 3V14, 3V15, 3V16, 3V2, 3V3, 3V4, 3V5, 3V6, 3V7, 3V8, 3V9: JUMPER-SMT_2_NC_TRACE_SILK, SparkFun-Jumpers:SMT-JUMPER_2_NC_TRACE_SILK
- added D1, D10, D11, D12, D13, D14, D15, D16, D2, D3, D4, D5, D6, D7, D8, D9: RED, SparkFun-LED:LED-0603
- added E$4: (no value), SparkFun-Aesthetics:FIDUCIAL-1X2
- added E$5: (no value), SparkFun-Retired:FIDUCIAL-1.5X3
- added R100, R101, R102, R103, R106, R107, R108, R109, R110, R99: 2.2k, SparkFun-Resistors:0603
- added R104, R111, R97: 10k, SparkFun-Resistors:0603
- added R105, R112, R98: 1k, SparkFun-Resistors:0603
- added U$577, U$617: (no value), buzzard_labels (52):#INT0
- added U$578, U$618: (no value), buzzard_labels (54):#INT0
- added U$579, U$619: (no value), buzzard_labels (60):QWIIC1
- added U$580, U$620: (no value), buzzard_labels (61):GPIO1
- added U$581, U$621: (no value), buzzard_labels (5):04
- added U$582, U$622: (no value), buzzard_labels (5):15
- added U$583, U$623: (no value), buzzard_labels (5):20
- added U$584, U$624: (no value), buzzard_labels (5):31
- added U$585, U$625: (no value), buzzard_labels (5):GND2
- added U$586, U$626: (no value), buzzard_labels (5):3V33
- added U$587, U$627: (no value), buzzard_labels (62):3V32
- added U$588, U$628: (no value), buzzard_labels (62):GND1
- added U$589, U$590, U$629, U$630: (no value), buzzard_labels (66):INT1
- added U$591, U$592, U$631, U$632: (no value), buzzard_labels (66):PWR0
- added U$593, U$633: (no value), buzzard_labels (68):____0____1
- added U$594, U$634: (no value), buzzard_labels (68):____2____3
- added U$595, U$635: (no value), buzzard_labels (68):____3____4
- added U$596, U$636: (no value), buzzard_labels (68):_____1____2
- added U$597, U$598, U$637, U$638: (no value), buzzard_labels (68):GND0
- added U$599, U$600, U$639, U$640: (no value), buzzard_labels (71):_3V3_0
- added U$601, U$602: SPARKX-LOGO3, SparkX:SPARKX-SMALL
- added U$603, U$616: (no value), buzzard_labels (44):3V33
- added U$604: (no value), buzzard_labels (44):A11
- added U$605, U$615: (no value), buzzard_labels (44):GND4
- added U$606: (no value), buzzard_labels (44):QWIIC_GPIO7
- added U$607: (no value), buzzard_labels (44):SCL6
- added U$608: (no value), buzzard_labels (44):SDA5
- added U$609: (no value), buzzard_labels (45):A00
- added U$610: (no value), buzzard_labels (45):A21
- added U$611: (no value), Labels:I_SUPER2_C-()-03
- added U$612: (no value), SparkFun-Aesthetics:QWIIC_6MM
- added U$613: (no value), buzzard_labels (51):SCL0
- added U$614: (no value), buzzard_labels (51):SDA1
- E$3: device SparkFun-Retired:FIDUCIAL-1.5X3 -> SparkFun-Aesthetics:FIDUCIAL-1X2
- R12, R18, R24, R30, R36, R54, R60, R66, R72, R78, R96: value 10k -> 2.2k
- R13, R20, R27, R34, R41, R55, R62, R69, R76, R83: value 2.2k -> 10k
- R14, R21, R28, R35, R49, R56, R63, R7, R70, R77, R91: value 2.2k -> 1k
- R42, R84: value 10k -> 1k
- U$109, U$110, U$30, U$31, U$469, U$470: value SPARKX-LOGO3 -> (none); device SparkX:SPARKX-SMALL -> buzzard_labels (66):INT1
- U$111, U$312, U$39, U$471: device buzzard_labels (44):3V33 -> buzzard_labels (66):PWR0
- U$112, U$40, U$472: device buzzard_labels (44):A11 -> buzzard_labels (66):PWR0
- U$113, U$41, U$473: device buzzard_labels (44):GND4 -> buzzard_labels (68):____0____1
- U$114, U$42, U$474: device buzzard_labels (44):QWIIC_GPIO7 -> buzzard_labels (68):____2____3
- U$115, U$43, U$475: device buzzard_labels (44):SCL6 -> buzzard_labels (68):____3____4
- U$116, U$44, U$476: device buzzard_labels (44):SDA5 -> buzzard_labels (68):_____1____2
- U$117, U$45, U$477: device buzzard_labels (45):A00 -> buzzard_labels (68):GND0
- U$118, U$46, U$478: device buzzard_labels (45):A21 -> buzzard_labels (68):GND0
- U$119, U$160, U$47, U$479, U$520: device buzzard_labels (47):__3V3__3 -> buzzard_labels (71):_3V3_0
- U$120, U$159, U$48, U$480, U$519: device buzzard_labels (48):__GND__0 -> buzzard_labels (71):_3V3_0
- U$121, U$481: value (none) -> SPARKX-LOGO3; device buzzard_labels (48):_____3_____2 -> SparkX:SPARKX-SMALL
- U$122, U$482: value (none) -> SPARKX-LOGO3; device buzzard_labels (48):______2______1 -> SparkX:SPARKX-SMALL
- U$123, U$336, U$483: device buzzard_labels (48):__GND__0 -> buzzard_labels (44):3V33
- U$124, U$15, U$484: device buzzard_labels (47):__3V3__3 -> buzzard_labels (44):A11
- U$125, U$16, U$485: device buzzard_labels (49):_____1_____1 -> buzzard_labels (44):GND4
- U$126, U$17, U$486: device buzzard_labels (49):______0______0 -> buzzard_labels (44):QWIIC_GPIO7
- U$127, U$487: device Labels:I_SUPER2_C-()-03 -> buzzard_labels (44):SCL6
- U$128, U$488: device SparkFun-Aesthetics:QWIIC_6MM -> buzzard_labels (44):SDA5
- U$129, U$489: device buzzard_labels (51):SCL0 -> buzzard_labels (45):A00
- U$130, U$490: device buzzard_labels (51):SDA1 -> buzzard_labels (45):A21
- U$131, U$491: device buzzard_labels (44):GND4 -> Labels:I_SUPER2_C-()-03
- U$132, U$492: device buzzard_labels (44):3V33 -> SparkFun-Aesthetics:QWIIC_6MM
- U$133, U$493: device buzzard_labels (52):#INT0 -> buzzard_labels (51):SCL0
- U$134, U$494: device buzzard_labels (54):#INT0 -> buzzard_labels (51):SDA1
- U$135, U$495: device buzzard_labels (60):QWIIC1 -> buzzard_labels (44):GND4
- U$136, U$496: device buzzard_labels (61):GPIO1 -> buzzard_labels (44):3V33
- U$137, U$497: device buzzard_labels (5):04 -> buzzard_labels (52):#INT0
- U$138, U$498: device buzzard_labels (5):15 -> buzzard_labels (54):#INT0
- U$139, U$499: device buzzard_labels (5):20 -> buzzard_labels (60):QWIIC1
- U$14, U$376, U$443, U$83: device buzzard_labels (47):__3V3__3 -> buzzard_labels (44):3V33
- U$140, U$500: device buzzard_labels (5):31 -> buzzard_labels (61):GPIO1
- U$141, U$501: device buzzard_labels (5):GND2 -> buzzard_labels (5):04
- U$142, U$502: device buzzard_labels (5):3V33 -> buzzard_labels (5):15
- U$143, U$503: device buzzard_labels (62):3V32 -> buzzard_labels (5):20
- U$144, U$504: device buzzard_labels (62):GND1 -> buzzard_labels (5):31
- U$145, U$505: value SPARKX-LOGO3 -> (none); device SparkX:SPARKX-SMALL -> buzzard_labels (5):GND2
- U$146, U$506: value SPARKX-LOGO3 -> (none); device SparkX:SPARKX-SMALL -> buzzard_labels (5):3V33
- U$147, U$507: device buzzard_labels (44):3V33 -> buzzard_labels (62):3V32
- U$148, U$508: device buzzard_labels (44):A11 -> buzzard_labels (62):GND1
- U$149, U$509: device buzzard_labels (44):GND4 -> buzzard_labels (66):INT1
- U$150, U$510: device buzzard_labels (44):QWIIC_GPIO7 -> buzzard_labels (66):INT1
- U$151, U$511: device buzzard_labels (44):SCL6 -> buzzard_labels (66):PWR0
- U$152, U$512: device buzzard_labels (44):SDA5 -> buzzard_labels (66):PWR0
- U$153, U$513: device buzzard_labels (45):A00 -> buzzard_labels (68):____0____1
- U$154, U$514: device buzzard_labels (45):A21 -> buzzard_labels (68):____2____3
- U$155, U$515: device buzzard_labels (47):__3V3__3 -> buzzard_labels (68):____3____4
- U$156, U$516: device buzzard_labels (48):__GND__0 -> buzzard_labels (68):_____1____2
- U$157, U$517: device buzzard_labels (48):_____3_____2 -> buzzard_labels (68):GND0
- U$158, U$518: device buzzard_labels (48):______2______1 -> buzzard_labels (68):GND0
- U$161, U$521: value (none) -> SPARKX-LOGO3; device buzzard_labels (49):_____1_____1 -> SparkX:SPARKX-SMALL
- U$162, U$522: value (none) -> SPARKX-LOGO3; device buzzard_labels (49):______0______0 -> SparkX:SPARKX-SMALL
- U$163, U$523: device Labels:I_SUPER2_C-()-03 -> buzzard_labels (44):3V33
- U$164, U$524: device SparkFun-Aesthetics:QWIIC_6MM -> buzzard_labels (44):A11
- U$165, U$525: device buzzard_labels (51):SCL0 -> buzzard_labels (44):GND4
- U$166, U$526: device buzzard_labels (51):SDA1 -> buzzard_labels (44):QWIIC_GPIO7
- U$167, U$527: device buzzard_labels (44):GND4 -> buzzard_labels (44):SCL6
- U$168, U$528: device buzzard_labels (44):3V33 -> buzzard_labels (44):SDA5
- U$169, U$529: device buzzard_labels (52):#INT0 -> buzzard_labels (45):A00
- U$170, U$530: device buzzard_labels (54):#INT0 -> buzzard_labels (45):A21
- U$171, U$531: device buzzard_labels (60):QWIIC1 -> Labels:I_SUPER2_C-()-03
- U$172, U$532: device buzzard_labels (61):GPIO1 -> SparkFun-Aesthetics:QWIIC_6MM
- U$173, U$533: device buzzard_labels (5):04 -> buzzard_labels (51):SCL0
- U$174, U$534: device buzzard_labels (5):15 -> buzzard_labels (51):SDA1
- U$175, U$535: device buzzard_labels (5):20 -> buzzard_labels (44):GND4
- U$176, U$536: device buzzard_labels (5):31 -> buzzard_labels (44):3V33
- U$177, U$537: device buzzard_labels (5):GND2 -> buzzard_labels (52):#INT0
- U$178, U$538: device buzzard_labels (5):3V33 -> buzzard_labels (54):#INT0
- U$179, U$539: device buzzard_labels (62):3V32 -> buzzard_labels (60):QWIIC1
- U$18: device buzzard_labels (48):_____3_____2 -> buzzard_labels (44):SCL6
- U$180, U$540: device buzzard_labels (62):GND1 -> buzzard_labels (61):GPIO1
- U$181, U$541: value SPARKX-LOGO3 -> (none); device SparkX:SPARKX-SMALL -> buzzard_labels (5):04
- U$182, U$542: value SPARKX-LOGO3 -> (none); device SparkX:SPARKX-SMALL -> buzzard_labels (5):15
- U$183, U$543: device buzzard_labels (44):3V33 -> buzzard_labels (5):20
- U$184, U$544: device buzzard_labels (44):A11 -> buzzard_labels (5):31
- U$185, U$545: device buzzard_labels (44):GND4 -> buzzard_labels (5):GND2
- U$186, U$546: device buzzard_labels (44):QWIIC_GPIO7 -> buzzard_labels (5):3V33
- U$187, U$547: device buzzard_labels (44):SCL6 -> buzzard_labels (62):3V32
- U$188, U$548: device buzzard_labels (44):SDA5 -> buzzard_labels (62):GND1
- U$189, U$549: device buzzard_labels (45):A00 -> buzzard_labels (66):INT1
- U$19: device buzzard_labels (48):______2______1 -> buzzard_labels (44):SDA5
- U$190, U$550: device buzzard_labels (45):A21 -> buzzard_labels (66):INT1
- U$191, U$232, U$551: device buzzard_labels (47):__3V3__3 -> buzzard_labels (66):PWR0
- U$192, U$231, U$552: device buzzard_labels (48):__GND__0 -> buzzard_labels (66):PWR0
- U$193, U$553: device buzzard_labels (48):_____3_____2 -> buzzard_labels (68):____0____1
- U$194, U$554: device buzzard_labels (48):______2______1 -> buzzard_labels (68):____2____3
- U$195, U$555: device buzzard_labels (48):__GND__0 -> buzzard_labels (68):____3____4
- U$196, U$556: device buzzard_labels (47):__3V3__3 -> buzzard_labels (68):_____1____2
- U$197, U$557: device buzzard_labels (49):_____1_____1 -> buzzard_labels (68):GND0
- U$198, U$558: device buzzard_labels (49):______0______0 -> buzzard_labels (68):GND0
- U$199, U$559: device Labels:I_SUPER2_C-()-03 -> buzzard_labels (71):_3V3_0
- U$200, U$560: device SparkFun-Aesthetics:QWIIC_6MM -> buzzard_labels (71):_3V3_0
- U$201, U$561: value (none) -> SPARKX-LOGO3; device buzzard_labels (51):SCL0 -> SparkX:SPARKX-SMALL
- U$202, U$562: value (none) -> SPARKX-LOGO3; device buzzard_labels (51):SDA1 -> SparkX:SPARKX-SMALL
- U$203, U$563: device buzzard_labels (44):GND4 -> buzzard_labels (44):3V33
- U$204, U$564: device buzzard_labels (44):3V33 -> buzzard_labels (44):A11
- U$205, U$565: device buzzard_labels (52):#INT0 -> buzzard_labels (44):GND4
- U$206, U$566: device buzzard_labels (54):#INT0 -> buzzard_labels (44):QWIIC_GPIO7
- U$207, U$567: device buzzard_labels (60):QWIIC1 -> buzzard_labels (44):SCL6
- U$208, U$568: device buzzard_labels (61):GPIO1 -> buzzard_labels (44):SDA5
- U$209, U$569: device buzzard_labels (5):04 -> buzzard_labels (45):A00
- U$210, U$570: device buzzard_labels (5):15 -> buzzard_labels (45):A21
- U$211, U$571: device buzzard_labels (5):20 -> Labels:I_SUPER2_C-()-03
- U$212, U$572: device buzzard_labels (5):31 -> SparkFun-Aesthetics:QWIIC_6MM
- U$213, U$573: device buzzard_labels (5):GND2 -> buzzard_labels (51):SCL0
- U$214, U$574: device buzzard_labels (5):3V33 -> buzzard_labels (51):SDA1
- U$215, U$575: device buzzard_labels (62):3V32 -> buzzard_labels (44):GND4
- U$216, U$576: device buzzard_labels (62):GND1 -> buzzard_labels (44):3V33
- U$217: value SPARKX-LOGO3 -> (none); device SparkX:SPARKX-SMALL -> buzzard_labels (52):#INT0
- U$218: value SPARKX-LOGO3 -> (none); device SparkX:SPARKX-SMALL -> buzzard_labels (54):#INT0
- U$219: device buzzard_labels (44):3V33 -> buzzard_labels (60):QWIIC1
- U$220: device buzzard_labels (44):A11 -> buzzard_labels (61):GPIO1
- U$221: device buzzard_labels (44):GND4 -> buzzard_labels (5):04
- U$222: device buzzard_labels (44):QWIIC_GPIO7 -> buzzard_labels (5):15
- U$223: device buzzard_labels (44):SCL6 -> buzzard_labels (5):20
- U$224: device buzzard_labels (44):SDA5 -> buzzard_labels (5):31
- U$225: device buzzard_labels (45):A00 -> buzzard_labels (5):GND2
- U$226: device buzzard_labels (45):A21 -> buzzard_labels (5):3V33
- U$227: device buzzard_labels (47):__3V3__3 -> buzzard_labels (62):3V32
- U$228: device buzzard_labels (48):__GND__0 -> buzzard_labels (62):GND1
- U$229: device buzzard_labels (48):_____3_____2 -> buzzard_labels (66):INT1
- U$230: device buzzard_labels (48):______2______1 -> buzzard_labels (66):INT1
- U$233: device buzzard_labels (49):_____1_____1 -> buzzard_labels (68):____0____1
- U$234: device buzzard_labels (49):______0______0 -> buzzard_labels (68):____2____3
- U$235: device Labels:I_SUPER2_C-()-03 -> buzzard_labels (68):____3____4
- U$236: device SparkFun-Aesthetics:QWIIC_6MM -> buzzard_labels (68):_____1____2
- U$237: device buzzard_labels (51):SCL0 -> buzzard_labels (68):GND0
- U$238: device buzzard_labels (51):SDA1 -> buzzard_labels (68):GND0
- U$239: device buzzard_labels (44):GND4 -> buzzard_labels (71):_3V3_0
- U$240, U$399: device buzzard_labels (44):3V33 -> buzzard_labels (71):_3V3_0
- U$241: value (none) -> SPARKX-LOGO3; device buzzard_labels (52):#INT0 -> SparkX:SPARKX-SMALL
- U$242: value (none) -> SPARKX-LOGO3; device buzzard_labels (54):#INT0 -> SparkX:SPARKX-SMALL
- U$243: device buzzard_labels (60):QWIIC1 -> buzzard_labels (44):3V33
- U$244: device buzzard_labels (61):GPIO1 -> buzzard_labels (44):A11
- U$245: device buzzard_labels (5):04 -> buzzard_labels (44):GND4
- U$246: device buzzard_labels (5):15 -> buzzard_labels (44):QWIIC_GPIO7
- U$247: device buzzard_labels (5):20 -> buzzard_labels (44):SCL6
- U$248: device buzzard_labels (5):31 -> buzzard_labels (44):SDA5
- U$249: device buzzard_labels (5):GND2 -> buzzard_labels (45):A00
- U$250: device buzzard_labels (5):3V33 -> buzzard_labels (45):A21
- U$251: device buzzard_labels (62):3V32 -> Labels:I_SUPER2_C-()-03
- U$252: device buzzard_labels (62):GND1 -> SparkFun-Aesthetics:QWIIC_6MM
- U$253: value SPARKX-LOGO3 -> (none); device SparkX:SPARKX-SMALL -> buzzard_labels (51):SCL0
- U$254: value SPARKX-LOGO3 -> (none); device SparkX:SPARKX-SMALL -> buzzard_labels (51):SDA1
- U$255: device buzzard_labels (44):3V33 -> buzzard_labels (44):GND4
- U$256: device buzzard_labels (44):A11 -> buzzard_labels (44):3V33
- U$257: device buzzard_labels (44):GND4 -> buzzard_labels (52):#INT0
- U$258: device buzzard_labels (44):QWIIC_GPIO7 -> buzzard_labels (54):#INT0
- U$259: device buzzard_labels (44):SCL6 -> buzzard_labels (60):QWIIC1
- U$260: device buzzard_labels (44):SDA5 -> buzzard_labels (61):GPIO1
- U$261: device buzzard_labels (45):A00 -> buzzard_labels (5):04
- U$262: device buzzard_labels (45):A21 -> buzzard_labels (5):15
- U$263: device buzzard_labels (47):__3V3__3 -> buzzard_labels (5):20
- U$264: device buzzard_labels (48):__GND__0 -> buzzard_labels (5):31
- U$265: device buzzard_labels (48):_____3_____2 -> buzzard_labels (5):GND2
- U$266: device buzzard_labels (48):______2______1 -> buzzard_labels (5):3V33
- U$267: device buzzard_labels (48):__GND__0 -> buzzard_labels (62):3V32
- U$268: device buzzard_labels (47):__3V3__3 -> buzzard_labels (62):GND1
- U$269: device buzzard_labels (49):_____1_____1 -> buzzard_labels (66):INT1
- U$270: device buzzard_labels (49):______0______0 -> buzzard_labels (66):INT1
- U$271: device Labels:I_SUPER2_C-()-03 -> buzzard_labels (66):PWR0
- U$272: device SparkFun-Aesthetics:QWIIC_6MM -> buzzard_labels (66):PWR0
- U$273: device buzzard_labels (51):SCL0 -> buzzard_labels (68):____0____1
- U$274: device buzzard_labels (51):SDA1 -> buzzard_labels (68):____2____3
- U$275: device buzzard_labels (44):GND4 -> buzzard_labels (68):____3____4
- U$276: device buzzard_labels (44):3V33 -> buzzard_labels (68):_____1____2
- U$277: device buzzard_labels (52):#INT0 -> buzzard_labels (68):GND0
- U$278: device buzzard_labels (54):#INT0 -> buzzard_labels (68):GND0
- U$279: device buzzard_labels (60):QWIIC1 -> buzzard_labels (71):_3V3_0
- U$280: device buzzard_labels (61):GPIO1 -> buzzard_labels (71):_3V3_0
- U$281: value (none) -> SPARKX-LOGO3; device buzzard_labels (5):04 -> SparkX:SPARKX-SMALL
- U$282: value (none) -> SPARKX-LOGO3; device buzzard_labels (5):15 -> SparkX:SPARKX-SMALL
- U$283: device buzzard_labels (5):20 -> buzzard_labels (44):3V33
- U$284: device buzzard_labels (5):31 -> buzzard_labels (44):A11
- U$285: device buzzard_labels (5):GND2 -> buzzard_labels (44):GND4
- U$286: device buzzard_labels (5):3V33 -> buzzard_labels (44):QWIIC_GPIO7
- U$287: device buzzard_labels (62):3V32 -> buzzard_labels (44):SCL6
- U$288: device buzzard_labels (62):GND1 -> buzzard_labels (44):SDA5
- U$289: value SPARKX-LOGO3 -> (none); device SparkX:SPARKX-SMALL -> buzzard_labels (45):A00
- U$290: value SPARKX-LOGO3 -> (none); device SparkX:SPARKX-SMALL -> buzzard_labels (45):A21
- U$291: device buzzard_labels (44):3V33 -> Labels:I_SUPER2_C-()-03
- U$292: device buzzard_labels (44):A11 -> SparkFun-Aesthetics:QWIIC_6MM
- U$293: device buzzard_labels (44):GND4 -> buzzard_labels (51):SCL0
- U$294: device buzzard_labels (44):QWIIC_GPIO7 -> buzzard_labels (51):SDA1
- U$295: device buzzard_labels (44):SCL6 -> buzzard_labels (44):GND4
- U$296: device buzzard_labels (44):SDA5 -> buzzard_labels (44):3V33
- U$297: device buzzard_labels (45):A00 -> buzzard_labels (52):#INT0
- U$298: device buzzard_labels (45):A21 -> buzzard_labels (54):#INT0
- U$299: device buzzard_labels (47):__3V3__3 -> buzzard_labels (60):QWIIC1
- U$300: device buzzard_labels (48):__GND__0 -> buzzard_labels (61):GPIO1
- U$301: device buzzard_labels (48):_____3_____2 -> buzzard_labels (5):04
- U$302: device buzzard_labels (48):______2______1 -> buzzard_labels (5):15
- U$303: device buzzard_labels (48):__GND__0 -> buzzard_labels (5):20
- U$304: device buzzard_labels (47):__3V3__3 -> buzzard_labels (5):31
- U$305: device buzzard_labels (49):_____1_____1 -> buzzard_labels (5):GND2
- U$306: device buzzard_labels (49):______0______0 -> buzzard_labels (5):3V33
- U$307: device Labels:I_SUPER2_C-()-03 -> buzzard_labels (62):3V32
- U$308: device SparkFun-Aesthetics:QWIIC_6MM -> buzzard_labels (62):GND1
- U$309: device buzzard_labels (51):SCL0 -> buzzard_labels (66):INT1
- U$310: device buzzard_labels (51):SDA1 -> buzzard_labels (66):INT1
- U$311: device buzzard_labels (44):GND4 -> buzzard_labels (66):PWR0
- U$313: device buzzard_labels (52):#INT0 -> buzzard_labels (68):____0____1
- U$314: device buzzard_labels (54):#INT0 -> buzzard_labels (68):____2____3
- U$315: device buzzard_labels (60):QWIIC1 -> buzzard_labels (68):____3____4
- U$316: device buzzard_labels (61):GPIO1 -> buzzard_labels (68):_____1____2
- U$317: device buzzard_labels (5):04 -> buzzard_labels (68):GND0
- U$318: device buzzard_labels (5):15 -> buzzard_labels (68):GND0
- U$319: device buzzard_labels (5):20 -> buzzard_labels (71):_3V3_0
- U$320: device buzzard_labels (5):31 -> buzzard_labels (71):_3V3_0
- U$321: value (none) -> SPARKX-LOGO3; device buzzard_labels (5):GND2 -> SparkX:SPARKX-SMALL
- U$322: value (none) -> SPARKX-LOGO3; device buzzard_labels (5):3V33 -> SparkX:SPARKX-SMALL
- U$323: device buzzard_labels (62):3V32 -> buzzard_labels (44):3V33
- U$324: device buzzard_labels (62):GND1 -> buzzard_labels (44):A11
- U$325: value SPARKX-LOGO3 -> (none); device SparkX:SPARKX-SMALL -> buzzard_labels (44):GND4
- U$326: value SPARKX-LOGO3 -> (none); device SparkX:SPARKX-SMALL -> buzzard_labels (44):QWIIC_GPIO7
- U$327: device buzzard_labels (44):3V33 -> buzzard_labels (44):SCL6
- U$328: device buzzard_labels (44):A11 -> buzzard_labels (44):SDA5
- U$329: device buzzard_labels (44):GND4 -> buzzard_labels (45):A00
- U$330: device buzzard_labels (44):QWIIC_GPIO7 -> buzzard_labels (45):A21
- U$331: device buzzard_labels (44):SCL6 -> Labels:I_SUPER2_C-()-03
- U$332: device buzzard_labels (44):SDA5 -> SparkFun-Aesthetics:QWIIC_6MM
- U$333: device buzzard_labels (45):A00 -> buzzard_labels (51):SCL0
- U$334: device buzzard_labels (45):A21 -> buzzard_labels (51):SDA1
- U$335: device buzzard_labels (47):__3V3__3 -> buzzard_labels (44):GND4
- U$337: device buzzard_labels (48):_____3_____2 -> buzzard_labels (52):#INT0
- U$338: device buzzard_labels (48):______2______1 -> buzzard_labels (54):#INT0
- U$339: device buzzard_labels (48):__GND__0 -> buzzard_labels (60):QWIIC1
- U$340: device buzzard_labels (47):__3V3__3 -> buzzard_labels (61):GPIO1
- U$341: device buzzard_labels (49):_____1_____1 -> buzzard_labels (5):04
- U$342: device buzzard_labels (49):______0______0 -> buzzard_labels (5):15
- U$343: device Labels:I_SUPER2_C-()-03 -> buzzard_labels (5):20
- U$344: device SparkFun-Aesthetics:QWIIC_6MM -> buzzard_labels (5):31
- U$345: device buzzard_labels (51):SCL0 -> buzzard_labels (5):GND2
- U$346: device buzzard_labels (51):SDA1 -> buzzard_labels (5):3V33
- U$347: device buzzard_labels (44):GND4 -> buzzard_labels (62):3V32
- U$348: device buzzard_labels (44):3V33 -> buzzard_labels (62):GND1
- U$349: device buzzard_labels (52):#INT0 -> buzzard_labels (66):INT1
- U$350: device buzzard_labels (54):#INT0 -> buzzard_labels (66):INT1
- U$351: device buzzard_labels (60):QWIIC1 -> buzzard_labels (66):PWR0
- U$352: device buzzard_labels (61):GPIO1 -> buzzard_labels (66):PWR0
- U$353: device buzzard_labels (5):04 -> buzzard_labels (68):____0____1
- U$354: device buzzard_labels (5):15 -> buzzard_labels (68):____2____3
- U$355: device buzzard_labels (5):20 -> buzzard_labels (68):____3____4
- U$356: device buzzard_labels (5):31 -> buzzard_labels (68):_____1____2
- U$357: device buzzard_labels (5):GND2 -> buzzard_labels (68):GND0
- U$358: device buzzard_labels (5):3V33 -> buzzard_labels (68):GND0
- U$359: device buzzard_labels (62):3V32 -> buzzard_labels (71):_3V3_0
- U$360: device buzzard_labels (62):GND1 -> buzzard_labels (71):_3V3_0
- U$371: device buzzard_labels (47):__3V3__3 -> Labels:I_SUPER2_C-()-03
- U$372: device buzzard_labels (48):__GND__0 -> SparkFun-Aesthetics:QWIIC_6MM
- U$373: device buzzard_labels (48):_____3_____2 -> buzzard_labels (51):SCL0
- U$374: device buzzard_labels (48):______2______1 -> buzzard_labels (51):SDA1
- U$375: device buzzard_labels (48):__GND__0 -> buzzard_labels (44):GND4
- U$377: device buzzard_labels (49):_____1_____1 -> buzzard_labels (52):#INT0
- U$378: device buzzard_labels (49):______0______0 -> buzzard_labels (54):#INT0
- U$379: device Labels:I_SUPER2_C-()-03 -> buzzard_labels (60):QWIIC1
- U$380: device SparkFun-Aesthetics:QWIIC_6MM -> buzzard_labels (61):GPIO1
- U$381: device buzzard_labels (51):SCL0 -> buzzard_labels (5):04
- U$382: device buzzard_labels (51):SDA1 -> buzzard_labels (5):15
- U$383: device buzzard_labels (44):GND4 -> buzzard_labels (5):20
- U$384: device buzzard_labels (44):3V33 -> buzzard_labels (5):31
- U$385: device buzzard_labels (52):#INT0 -> buzzard_labels (5):GND2
- U$386: device buzzard_labels (54):#INT0 -> buzzard_labels (5):3V33
- U$387: device buzzard_labels (60):QWIIC1 -> buzzard_labels (62):3V32
- U$388: device buzzard_labels (61):GPIO1 -> buzzard_labels (62):GND1
- U$389: device buzzard_labels (5):04 -> buzzard_labels (66):INT1
- U$390: device buzzard_labels (5):15 -> buzzard_labels (66):INT1
- U$391: device buzzard_labels (5):20 -> buzzard_labels (66):PWR0
- U$392: device buzzard_labels (5):31 -> buzzard_labels (66):PWR0
- U$393: device buzzard_labels (5):GND2 -> buzzard_labels (68):____0____1
- U$394: device buzzard_labels (5):3V33 -> buzzard_labels (68):____2____3
- U$395: device buzzard_labels (62):3V32 -> buzzard_labels (68):____3____4
- U$396: device buzzard_labels (62):GND1 -> buzzard_labels (68):_____1____2
- U$397, U$398: value SPARKX-LOGO3 -> (none); device SparkX:SPARKX-SMALL -> buzzard_labels (68):GND0
- U$4, U$6: value (none) -> SPARKX-LOGO3; device buzzard_labels (48):__GND__0 -> SparkX:SPARKX-SMALL
- U$400: device buzzard_labels (44):A11 -> buzzard_labels (71):_3V3_0
- U$401: value (none) -> SPARKX-LOGO3; device buzzard_labels (44):GND4 -> SparkX:SPARKX-SMALL
- U$402: value (none) -> SPARKX-LOGO3; device buzzard_labels (44):QWIIC_GPIO7 -> SparkX:SPARKX-SMALL
- U$403: device buzzard_labels (44):SCL6 -> buzzard_labels (44):3V33
- U$404: device buzzard_labels (44):SDA5 -> buzzard_labels (44):A11
- U$405: device buzzard_labels (45):A00 -> buzzard_labels (44):GND4
- U$406: device buzzard_labels (45):A21 -> buzzard_labels (44):QWIIC_GPIO7
- U$407: device buzzard_labels (47):__3V3__3 -> buzzard_labels (44):SCL6
- U$408: device buzzard_labels (48):__GND__0 -> buzzard_labels (44):SDA5
- U$409, U$49: device buzzard_labels (48):_____3_____2 -> buzzard_labels (45):A00
- U$410, U$50: device buzzard_labels (48):______2______1 -> buzzard_labels (45):A21
- U$411, U$51: device buzzard_labels (48):__GND__0 -> Labels:I_SUPER2_C-()-03
- U$412, U$52: device buzzard_labels (47):__3V3__3 -> SparkFun-Aesthetics:QWIIC_6MM
- U$413, U$53: device buzzard_labels (49):_____1_____1 -> buzzard_labels (51):SCL0
- U$414, U$54: device buzzard_labels (49):______0______0 -> buzzard_labels (51):SDA1
- U$415, U$55: device Labels:I_SUPER2_C-()-03 -> buzzard_labels (44):GND4
- U$416, U$56: device SparkFun-Aesthetics:QWIIC_6MM -> buzzard_labels (44):3V33
- U$417, U$57: device buzzard_labels (51):SCL0 -> buzzard_labels (52):#INT0
- U$418, U$58: device buzzard_labels (51):SDA1 -> buzzard_labels (54):#INT0
- U$419, U$59: device buzzard_labels (44):GND4 -> buzzard_labels (60):QWIIC1
- U$420, U$60: device buzzard_labels (44):3V33 -> buzzard_labels (61):GPIO1
- U$421, U$61: device buzzard_labels (52):#INT0 -> buzzard_labels (5):04
- U$422, U$62: device buzzard_labels (54):#INT0 -> buzzard_labels (5):15
- U$423, U$63: device buzzard_labels (60):QWIIC1 -> buzzard_labels (5):20
- U$424, U$64: device buzzard_labels (61):GPIO1 -> buzzard_labels (5):31
- U$425, U$65: device buzzard_labels (5):04 -> buzzard_labels (5):GND2
- U$426, U$66: device buzzard_labels (5):15 -> buzzard_labels (5):3V33
- U$427, U$67: device buzzard_labels (5):20 -> buzzard_labels (62):3V32
- U$428, U$68: device buzzard_labels (5):31 -> buzzard_labels (62):GND1
- U$429, U$69: device buzzard_labels (5):GND2 -> buzzard_labels (66):INT1
- U$430, U$70: device buzzard_labels (5):3V33 -> buzzard_labels (66):INT1
- U$431, U$71: device buzzard_labels (62):3V32 -> buzzard_labels (66):PWR0
- U$432, U$72: device buzzard_labels (62):GND1 -> buzzard_labels (66):PWR0
- U$433, U$73: value SPARKX-LOGO3 -> (none); device SparkX:SPARKX-SMALL -> buzzard_labels (68):____0____1
- U$434, U$74: value SPARKX-LOGO3 -> (none); device SparkX:SPARKX-SMALL -> buzzard_labels (68):____2____3
- U$435, U$75: device buzzard_labels (44):3V33 -> buzzard_labels (68):____3____4
- U$436, U$76: device buzzard_labels (44):A11 -> buzzard_labels (68):_____1____2
- U$437, U$77: device buzzard_labels (44):GND4 -> buzzard_labels (68):GND0
- U$438, U$78: device buzzard_labels (44):QWIIC_GPIO7 -> buzzard_labels (68):GND0
- U$439, U$79: device buzzard_labels (44):SCL6 -> buzzard_labels (71):_3V3_0
- U$440, U$80: device buzzard_labels (44):SDA5 -> buzzard_labels (71):_3V3_0
- U$441, U$81: value (none) -> SPARKX-LOGO3; device buzzard_labels (45):A00 -> SparkX:SPARKX-SMALL
- U$442, U$82: value (none) -> SPARKX-LOGO3; device buzzard_labels (45):A21 -> SparkX:SPARKX-SMALL
- U$444, U$84: device buzzard_labels (48):__GND__0 -> buzzard_labels (44):A11
- U$445, U$85: device buzzard_labels (48):_____3_____2 -> buzzard_labels (44):GND4
- U$446, U$86: device buzzard_labels (48):______2______1 -> buzzard_labels (44):QWIIC_GPIO7
- U$447, U$87: device buzzard_labels (48):__GND__0 -> buzzard_labels (44):SCL6
- U$448, U$88: device buzzard_labels (47):__3V3__3 -> buzzard_labels (44):SDA5
- U$449, U$89: device buzzard_labels (49):_____1_____1 -> buzzard_labels (45):A00
- U$450, U$90: device buzzard_labels (49):______0______0 -> buzzard_labels (45):A21
- moved E$3 209.6 mm to (147.0, 156.0)
- moved U$317 155.2 mm to (142.5, 37.6), flipped to the bottom
- moved R26 151.0 mm to (143.8, 14.0), turned to 180 degrees
- moved R25 147.8 mm to (143.8, 16.5), turned to 180 degrees
- moved U$447 147.6 mm to (147.8, 91.2), flipped to the top, turned to 0 degrees
- moved R54 145.8 mm to (143.8, 52.6), turned to 180 degrees
- moved E$2 145.3 mm to (6.86, 156.0), flipped to the bottom
- moved U$314 142.6 mm to (137.4, 37.1), turned to 90 degrees
- moved U$450 141.1 mm to (148.8, 98.8), turned to 0 degrees
- moved U$443 139.1 mm to (147.6, 86.1), flipped to the top, turned to 0 degrees
- moved U$449 138.4 mm to (148.8, 93.7), turned to 0 degrees
- moved U$319 137.7 mm to (142.4, 70.0), flipped to the bottom
- moved U$159 136.6 mm to (142.4, 31.4)
- moved U$448 134.9 mm to (147.6, 88.6), flipped to the top, turned to 0 degrees
- moved U$445 134.8 mm to (147.6, 83.6), flipped to the top, turned to 0 degrees
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Connections:
- new net N$17: D6.A, R42.1
- new net N$18: 3V6.1, R42.2
- new net N$19: JP60.1, R48.2
- new net N$20: D7.A, R49.1
- new net N$21: 3V7.1, R49.2
- new net N$22: JP69.1, R55.2
- new net N$23: D8.A, R56.1
- new net N$24: 3V8.1, R56.2
- new net N$25: JP78.1, R62.2
- new net N$26: D9.A, R63.1
- new net N$27: 3V9.1, R63.2
- new net N$28: JP87.1, R69.2
- new net N$29: D10.A, R70.1
- new net N$30: 3V10.1, R70.2
- new net N$31: JP96.1, R76.2
- new net N$32: D11.A, R77.1
- new net N$33: 3V11.1, R77.2
- new net N$34: JP105.1, R83.2
- new net N$35: D12.A, R84.1
- new net N$36: 3V12.1, R84.2
- new net N$37: JP114.1, R90.2
- new net N$38: D13.A, R91.1
- new net N$39: 3V13.1, R91.2
- new net N$40: JP123.1, R97.2
- new net N$41: D14.A, R98.1
- new net N$42: 3V14.1, R98.2
- new net N$43: JP132.1, R104.2
- new net N$44: D15.A, R105.1
- new net N$45: 3V15.1, R105.2
- new net N$46: JP141.1, R111.2
- new net N$47: D16.A, R112.1
- new net N$48: 3V16.1, R112.2
- net !INT1: now also R13.1; no longer R12.1
- net !INT10: now also R76.1; no longer R66.1
- net !INT11: now also R83.1; no longer R72.1
- net !INT12: now also R90.1; no longer R78.1
- net !INT13: now also R97.1; no longer R84.1
- net !INT14: now also R104.1; no longer R90.1
- net !INT15: now also R111.1; no longer R96.1
- net !INT2: now also R20.1; no longer R18.1
- net !INT3: now also R27.1; no longer R24.1
- net !INT4: now also R34.1; no longer R30.1
- net !INT5: now also R41.1; no longer R36.1
- net !INT6: now also R48.1; no longer R42.1
- net !INT7: now also R55.1; no longer R48.1
- net !INT8: now also R62.1; no longer R54.1
- net !INT9: now also R69.1; no longer R60.1
- net 3.3V: now also 3V3.2
- net 3.3V1: now also 3V1.2
- net 3.3V10: now also 3V11.2
- net 3.3V11: now also 3V12.2
- net 3.3V12: now also 3V13.2
- net 3.3V13: now also 3V14.2
- net 3.3V14: now also 3V15.2
- net 3.3V15: now also 3V16.2
- net 3.3V2: now also 3V2.2
- net 3.3V3: now also 3V4.2
- net 3.3V4: now also 3V5.2
- net 3.3V5: now also 3V6.2
- net 3.3V6: now also 3V7.2
- net 3.3V7: now also 3V8.2
- net 3.3V8: now also 3V9.2
- net 3.3V9: now also 3V10.2
- net A10: now also R25.2; no longer R22.2
- net A11: now also R24.2; no longer R21.2
- net A12: now also R33.2; no longer R29.2
- net A13: now also R32.2; no longer R28.2
- net A14: now also R31.2; no longer R27.2
- net A15: now also R40.2; no longer R35.2
- net A16: now also R39.2; no longer R34.2
- net A17: now also R38.2; no longer R33.2
- net A18: now also R47.2; no longer R41.2
- net A19: now also R46.2; no longer R40.2
- net A20: now also R45.2; no longer R39.2
- net A21: now also R54.2; no longer R47.2
- net A22: now also R53.2; no longer R46.2
- net A23: now also R52.2; no longer R45.2
- net A24: now also R61.2; no longer R53.2
- net A25: now also R60.2; no longer R52.2
- net A26: now also R59.2; no longer R51.2
- net A27: now also R68.2; no longer R59.2
- net A28: now also R67.2; no longer R58.2
- net A29: now also R66.2; no longer R57.2
- net A3: now also R12.2; no longer R11.2
- net A30: now also R75.2; no longer R65.2
- net A31: now also R74.2; no longer R64.2
- net A32: now also R73.2; no longer R63.2
- net A33: now also R82.2; no longer R71.2
- net A34: now also R81.2; no longer R70.2
- net A35: now also R80.2; no longer R69.2
- net A36: now also R89.2; no longer R77.2
- net A37: now also R88.2; no longer R76.2
- net A38: now also R87.2; no longer R75.2
- net A39: now also R96.2; no longer R83.2
- net A4: now also R11.2; no longer R10.2
- net A40: now also R95.2; no longer R82.2
- net A41: now also R94.2; no longer R81.2
- net A42: now also R103.2; no longer R89.2
- net A43: now also R102.2; no longer R88.2
- net A44: now also R101.2; no longer R87.2
- net A45: now also R110.2; no longer R95.2
- net A46: now also R109.2; no longer R94.2
- net A47: now also R108.2; no longer R93.2
- net A5: now also R10.2; no longer R9.2
- net A6: now also R19.2; no longer R17.2
- net A7: now also R18.2; no longer R16.2
- net A8: now also R17.2; no longer R15.2
- net A9: now also R26.2; no longer R23.2
- net GND: now also D1.C
- net GND1: now also D2.C, R12.1; no longer R9.1
- net GND10: now also D11.C, R73.1, R74.1, R75.1; no longer R63.1, R64.1, R65.1
- net GND11: now also D12.C, R80.1, R81.1, R82.1; no longer R69.1, R70.1, R71.1
- net GND12: now also D13.C, R87.1, R88.1, R89.1; no longer R75.1, R76.1, R77.1
- net GND13: now also D14.C, R94.1, R95.1, R96.1; no longer R81.1, R82.1, R83.1
- net GND14: now also D15.C, R101.1, R102.1, R103.1; no longer R87.1, R88.1, R89.1
- net GND15: now also D16.C, R108.1, R109.1, R110.1; no longer R93.1, R94.1, R95.1
- net GND2: now also D3.C, R18.1, R19.1; no longer R15.1, R16.1
- net GND3: now also D4.C, R24.1, R25.1, R26.1; no longer R21.1, R22.1, R23.1
- net GND4: now also D5.C, R31.1, R32.1, R33.1; no longer R27.1, R28.1, R29.1
- net GND5: now also D6.C, R38.1, R39.1, R40.1; no longer R33.1, R34.1, R35.1
- net GND6: now also D7.C, R45.1, R46.1, R47.1; no longer R39.1, R40.1, R41.1
- net GND7: now also D8.C, R52.1, R53.1, R54.1; no longer R45.1, R46.1, R47.1
- net GND8: now also D9.C, R59.1, R60.1, R61.1; no longer R51.1, R52.1, R53.1
- net GND9: now also D10.C, R66.1, R67.1, R68.1; no longer R57.1, R58.1, R59.1
- net N$10: now also JP33.1, R27.2; no longer JP87.1, R60.2
- net N$11: now also D4.A, R28.1; no longer JP96.1, R66.2
- net N$12: now also 3V4.1, R28.2; no longer JP105.1, R72.2
- net N$13: now also JP42.1, R34.2; no longer JP114.1, R78.2
- net N$14: now also D5.A, R35.1; no longer JP123.1, R84.2
- net N$15: now also 3V5.1, R35.2; no longer JP132.1, R90.2
- net N$16: now also JP51.1, R41.2; no longer JP141.1, R96.2
- net N$2: now also D1.A, R7.1; no longer JP15.1, R12.2
- net N$3: now also 3V3.1, R7.2; no longer JP24.1, R18.2
- net N$4: now also JP15.1, R13.2; no longer JP33.1, R24.2
- net N$5: now also D2.A, R14.1; no longer JP42.1, R30.2
- net N$6: now also 3V1.1, R14.2; no longer JP51.1, R36.2
- net N$7: now also JP24.1, R20.2; no longer JP60.1, R42.2
- net N$8: now also D3.A, R21.1; no longer JP69.1, R48.2
- net N$9: now also 3V2.1, R21.2; no longer JP78.1, R54.2
- net SCL1: now also R9.1; no longer R8.1
- net SCL10: now also R72.1; no longer R62.1
- net SCL11: now also R79.1; no longer R68.1
- net SCL12: now also R86.1; no longer R74.1
- net SCL13: now also R93.1; no longer R80.1
- net SCL14: now also R100.1; no longer R86.1
- net SCL15: now also R107.1; no longer R92.1
- net SCL2: now also R16.1; no longer R14.1
- net SCL3: now also R23.1; no longer R20.1
- net SCL4: now also R30.1; no longer R26.1
- net SCL5: now also R37.1; no longer R32.1
- net SCL6: now also R44.1; no longer R38.1
- net SCL7: now also R51.1; no longer R44.1
- net SCL8: now also R58.1; no longer R50.1
- net SCL9: now also R65.1; no longer R56.1
- net SCL_PU10: now also R64.2; no longer R55.2
- net SCL_PU11: now also R71.2; no longer R61.2
- net SCL_PU12: now also R78.2; no longer R67.2
- net SCL_PU13: now also R85.2; no longer R73.2
- net SCL_PU14: now also R92.2; no longer R79.2
- net SCL_PU15: now also R99.2; no longer R85.2
- net SCL_PU16: now also R106.2; no longer R91.2
- net SCL_PU2: now also R8.2; no longer R7.2
- net SCL_PU3: now also R15.2; no longer R13.2
- net SCL_PU4: now also R22.2; no longer R19.2
- net SCL_PU5: now also R29.2; no longer R25.2
- net SCL_PU6: now also R36.2; no longer R31.2
- net SCL_PU7: now also R43.2; no longer R37.2
- net SCL_PU8: now also R50.2; no longer R43.2
- net SCL_PU9: now also R57.2; no longer R49.2
- net SDA1: now also R8.1; no longer R7.1
- net SDA10: now also R71.1; no longer R61.1
- net SDA11: now also R78.1; no longer R67.1
- net SDA12: now also R85.1; no longer R73.1
- net SDA13: now also R92.1; no longer R79.1
- net SDA14: now also R99.1; no longer R85.1
- net SDA15: now also R106.1; no longer R91.1
- net SDA2: now also R15.1; no longer R13.1
- net SDA3: now also R22.1; no longer R19.1
- net SDA4: now also R29.1; no longer R25.1
- net SDA5: now also R36.1; no longer R31.1
- net SDA6: now also R43.1; no longer R37.1
- net SDA7: now also R50.1; no longer R43.1
- net SDA8: now also R57.1; no longer R49.1
- net SDA9: now also R64.1; no longer R55.1
- net SDA_PU10: now also R65.2; no longer R56.2
- net SDA_PU11: now also R72.2; no longer R62.2
- net SDA_PU12: now also R79.2; no longer R68.2
- net SDA_PU13: now also R86.2; no longer R74.2
- net SDA_PU14: now also R93.2; no longer R80.2
- net SDA_PU15: now also R100.2; no longer R86.2
- net SDA_PU16: now also R107.2; no longer R92.2
- net SDA_PU2: now also R9.2; no longer R8.2
- net SDA_PU3: now also R16.2; no longer R14.2
- net SDA_PU4: now also R23.2; no longer R20.2
- net SDA_PU5: now also R30.2; no longer R26.2
- net SDA_PU6: now also R37.2; no longer R32.2
- net SDA_PU7: now also R44.2; no longer R38.2
- net SDA_PU8: now also R51.2; no longer R44.2
- net SDA_PU9: now also R58.2; no longer R50.2
Routing:
- net N$40: track 0.00 -> 4.37 mm, vias 0 -> 1
- net N$37: track 0.00 -> 4.37 mm, vias 0 -> 1
- net N$28: track 0.00 -> 4.37 mm, vias 0 -> 1
- net N$25: track 0.00 -> 4.37 mm, vias 0 -> 1
- net N$46: track 0.00 -> 4.37 mm, vias 0 -> 1
- net N$43: track 0.00 -> 4.37 mm, vias 0 -> 1
- net N$34: track 0.00 -> 4.37 mm, vias 0 -> 1
- net N$31: track 0.00 -> 4.37 mm, vias 0 -> 1
- net N$22: track 0.00 -> 4.37 mm, vias 0 -> 1
- net N$19: track 0.00 -> 4.37 mm, vias 0 -> 1
- net N$36: track 0.00 -> 3.35 mm, vias 0 -> 1
- net N$24: track 0.00 -> 3.35 mm, vias 0 -> 1
- net N$27: track 0.00 -> 3.35 mm, vias 0 -> 1
- net N$18: track 0.00 -> 3.35 mm, vias 0 -> 1
- net N$30: track 0.00 -> 3.35 mm, vias 0 -> 1
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Other:
- board size 186.7 x 167.6 mm -> 174 x 174 mm
- board text removed: "Route Out"
